File: BNC-breakout/BNC-breakout.kicad_pcb (KiCad board)
At the start: 2 copper layers, 482.6 x 44.4 mm, 24 parts, among them J1 Conn_Coaxial, J10 Conn_Coaxial, J11 Conn_Coaxial, J12 Conn_Coaxial, J13 Conn_Coaxial, J14 Conn_Coaxial, J15 Conn_Coaxial, J16 Conn_Coaxial, J2 Conn_Coaxial, J3 Conn_Coaxial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

Commit message: 4-layer PCB. +V surrounded by GND
Parts:
- renumbered TP1 to +V, TP2 to GND
Routing:
- net +VSW: track 0.00 -> 405.0 mm
- added copper zone on In1.Cu, net +VSW
- added copper zone on F.Cu, net GND
- added copper zone on In2.Cu, net GND
- removed copper zone on F.Cu, net +VSW
Other:
- copper layers 2 -> 4
Changed lines of the file:
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@@
 	(layers
 		(0 "F.Cu" signal)
+		(4 "In1.Cu" signal)
+		(6 "In2.Cu" signal)
 		(2 "B.Cu" signal)
 		(9 "F.Adhes" user "F.Adhesive")
@@
 	)
 	(setup
+		(stackup
+			(layer "F.SilkS"
+				(type "Top Silk Screen")
+			)
+			(layer "F.Paste"
+				(type "Top Solder Paste")
+			)
+			(layer "F.Mask"
+				(type "Top Solder Mask")
+				(thickness 0.01)
+			)
+			(layer "F.Cu"
+				(type "copper")
+				(thickness 0.035)
+			)
+			(layer "dielectric 1"
+				(type "prepreg")
+				(thickness 0.1)
+				(material "FR4")
+				(epsilon_r 4.5)
+				(loss_tangent 0.02)
+			)
+			(layer "In1.Cu"
+				(type "copper")
+				(thickness 0.035)
+			)
+			(layer "dielectric 2"
+				(type "core")
+				(thickness 1.24)
+				(material "FR4")
+				(epsilon_r 4.5)
+				(loss_tangent 0.02)
+			)
+			(layer "In2.Cu"
+				(type "copper")
+				(thickness 0.035)
+			)
+			(layer "dielectric 3"
+				(type "prepreg")
+				(thickness 0.1)
+				(material "FR4")
+				(epsilon_r 4.5)
+				(loss_tangent 0.02)
+			)
+			(layer "B.Cu"
+				(type "copper")
+				(thickness 0.035)
+			)
+			(layer "B.Mask"
+				(type "Bottom Solder Mask")
+				(thickness 0.01)
+			)
+			(layer "B.Paste"
+				(type "Bottom Solder Paste")
+			)
+			(layer "B.SilkS"
+				(type "Bottom Silk Screen")
+			)
+			(copper_finish "None")
+			(dielectric_constraints no)
+		)
 		(pad_to_mask_clearance 0)
 		(allow_soldermask_bridges_in_footprints no)
@@
 		(descr "Soldered wire connection, for a single 4 mm² wire, reinforced insulation, conductor diameter 3mm, outer diameter 6mm, size source Multi-Contact FLEXI-xV 2.5 (https://www.staubli.com/content/dam/ecs/catalogs-brochures/TM/CAB-Main-11014119-en.pdf#page=11), bend radius 3 times outer diameter, generated with kicad-footprint-generator")
 		(tags "connector wire 4sqmm")
-		(property "Reference" "TP2"
+		(property "Reference" "GND"
 			(at 0 -4.2 0)
 			(layer "F.SilkS")
@@
 		(descr "Soldered wire connection, for a single 4 mm² wire, reinforced insulation, conductor diameter 3mm, outer diameter 6mm, size source Multi-Contact FLEXI-xV 2.5 (https://www.staubli.com/content/dam/ecs/catalogs-brochures/TM/CAB-Main-11014119-en.pdf#page=11), bend radius 3 times outer diameter, generated with kicad-footprint-generator")
 		(tags "connector wire 4sqmm")
-		(property "Reference" "TP1"
+		(property "Reference" "+V"
 			(at 0 -4.2 0)
 			(layer "F.SilkS")
@@
 		(layer "Edge.Cuts")
 	)
-	(zone
+	(segment
+		(start 63.5 47.625)
+		(end 444.5 47.625)
+		(width 1.5875)
+		(layer "In1.Cu")
 		(net 1)
-		(net_name "+VSW")
+	)
+	(segment
+		(start 42 41.5)
+		(end 48.125 47.625)
+		(width 1.5875)
+		(layer "In1.Cu")
+		(net 1)
+	)
+	(segment
+		(start 48.125 47.625)
+		(end 63.5 47.625)
+		(width 1.5875)
+		(layer "In1.Cu")
+		(net 1)
+	)
+	(zone
+		(net 2)
+		(net_name "GND")
 		(layer "F.Cu")
 		(hatch edge 0.5)
+		(priority 2)
 		(connect_pads
 			(clearance 0.5)
@@
 		(polygon
 			(pts
-				(xy 11 25) (xy 497 24) (xy 498.5 71) (xy 10.5 71)
+				(xy 11 24) (xy 500 23) (xy 500 73) (xy 12 74)
 			)
 		)
@@
 			)
 		)
+	)
+	(zone
+		(net 1)
+		(net_name "+VSW")
+		(layer "In1.Cu")
+		(hatch edge 0.5)
+		(connect_pads
+			(clearance 0.5)
+		)
+		(min_thickness 0.25)
+		(filled_areas_thickness no)
+		(fill yes
+			(thermal_gap 0.5)
+			(thermal_bridge_width 0.5)
+		)
+		(polygon
+			(pts
+				(xy 11 25) (xy 497 24) (xy 498.5 71) (xy 10.5 71)
+			)
+		)
+	)
+	(zone
+		(net 2)
+		(net_name "GND")
+		(layer "In2.Cu")
+		(hatch edge 0.5)
+		(priority 3)
+		(connect_pads
+			(clearance 0.5)
+		)
+		(min_thickness 0.25)
+		(filled_areas_thickness no)
+		(fill yes
+			(thermal_gap 0.5)
+			(thermal_bridge_width 0.5)
+		)
+		(polygon
+			(pts
+				(xy 10 23) (xy 501 22) (xy 501 75) (xy 11 73)
+			)
+		)
